File: LED_PANEL_26x45mm/LED_PANEL_26x45mm.kicad_pcb (KiCad board)
At the start: 2 copper layers, 51 x 32 mm, 4 parts

Commit message: pcb:(LED_PANEL)single gerber
Routing:
- added copper zone on B.Cu, net (none)
- added copper zone on F.Cu, net (none)
Changed lines of the file:
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@@
     (visible_elements FFFFFF7F)
     (pcbplotparams
-      (layerselection 0x010fc_ffffffff)
+      (layerselection 0x010f0_ffffffff)
       (usegerberextensions false)
       (usegerberattributes false)
@@
       (padsonsilk true)
       (subtractmaskfromsilk false)
-      (outputformat 5)
+      (outputformat 1)
       (mirror false)
-      (drillshape 1)
+      (drillshape 0)
       (scaleselection 1)
       (outputdirectory "gerber/single/"))
@@
   (gr_line (start 101 50) (end 101 82) (layer Edge.Cuts) (width 0.05))
   (gr_line (start 50 50) (end 50 82) (layer Edge.Cuts) (width 0.05))
+  (zone (net 0) (net_name "") (layer F.Cu) (hatch edge 0.508)
+    (connect_pads (clearance 0.508))
+    (min_thickness 0.254)
+    (fill yes (arc_segments 32) (thermal_gap 0.508) (thermal_bridge_width 0.508))
+    (polygon
+      (pts
+        (xy 102.79888 84.00288) (xy 49.0982 84.13496) (xy 49.23028 48.44288) (xy 76.55052 48.02124) (xy 103.06812 48.02124)
+      )
+    )
+  )
+  (zone (net 0) (net_name "") (layer B.Cu) (hatch edge 0.508)
+    (connect_pads (clearance 0.508))
+    (min_thickness 0.254)
+    (fill yes (arc_segments 32) (thermal_gap 0.508) (thermal_bridge_width 0.508))
+    (polygon
+      (pts
+        (xy 104.13492 84.70392) (xy 48.30064 84.56676) (xy 48.30064 47.75708) (xy 104.39908 46.89856)
+      )
+    )
+  )
 )
